Commit message: rename packages
Signed-off-by: Christopher Strøm <detoxte@gmail.com>

File: asv_description/urdf/accessories.urdf.xacro (robot description, xacro)
@@ -14,5 +14,5 @@
         <origin xyz="0 0 0" rpy="0 0 0" />
         <geometry>
-          <mesh filename="package://heron_vortex_description/meshes/${type}-rear-plate.stl"/>
+          <mesh filename="package://asv_description/meshes/${type}-rear-plate.stl"/>
         </geometry>
         <material name="dark_gray" />

File: asv_description/urdf/accessories/axis_ptz.urdf.xacro (robot description, xacro)
@@ -6,5 +6,5 @@
       <origin xyz="0 0 0" rpy="0 0 0" />
       <geometry>
-        <mesh filename="package://heron_vortex_description/meshes/axis_ptz.stl"/>
+        <mesh filename="package://asv_description/meshes/axis_ptz.stl"/>
       </geometry>
       <material name="axis_ptz_white">

File: asv_description/urdf/accessories/novatel_smart6.urdf.xacro (robot description, xacro)
@@ -6,5 +6,5 @@
       <origin xyz="0 0 0" rpy="0 0 0" />
       <geometry>
-        <mesh filename="package://heron_vortex_description/meshes/novatel-smart6.stl"/>
+        <mesh filename="package://asv_description/meshes/novatel-smart6.stl"/>
       </geometry>
       <material name="novatel_white">

File: asv_description/urdf/base.xacro (robot description, xacro)
@@ -10,5 +10,5 @@
   <xacro:property name="rho" value="1028"/>
   <!-- Loading vehicle's specific macros -->
-  <xacro:include filename="$(find heron_vortex_description)/urdf/snippets.xacro"/>
+  <xacro:include filename="$(find asv_description)/urdf/snippets.xacro"/>
   <material name="gray"><color rgba="0.7 0.7 0.7 1.0"/></material>
   <material name="dark_gray"><color rgba="0.2 0.2 0.2 1.0"/></material>
@@ -31,5 +31,5 @@
           <origin xyz="0 0 0" rpy="0 0 0" />
           <geometry>
-            <mesh filename="package://heron_vortex_description/meshes/${side}_panel.stl" />
+            <mesh filename="package://asv_description/meshes/${side}_panel.stl" />
           </geometry>
           <material name="yellow" />
@@ -51,5 +51,5 @@
           <origin xyz="0 0 0" rpy="0 0 0"/>
           <geometry>
-            <mesh filename="package://heron_vortex_description/meshes/heron_base.stl" scale="1 1 1" />
+            <mesh filename="package://asv_description/meshes/heron_base.stl" scale="1 1 1" />
           </geometry>
           <material name="dark_gray" />
@@ -58,5 +58,5 @@
           <origin xyz="0 0 0" rpy="0 0 0"/>
           <geometry>
-            <mesh filename="package://heron_vortex_description/meshes/heron_collision.stl" scale="1 1 1" />
+            <mesh filename="package://asv_description/meshes/heron_collision.stl" scale="1 1 1" />
           </geometry>
         </collision>
@@ -106,8 +106,8 @@
     </xacro:thruster_macro>
     <!-- Include the sensor modules -->
-    <xacro:include filename="$(find heron_vortex_description)/urdf/sensors.xacro"/>
+    <xacro:include filename="$(find asv_description)/urdf/sensors.xacro"/>
     <xacro:panel namespace="$(arg suffix_ns)" side="left" location="1" />
     <xacro:panel namespace="$(arg suffix_ns)" side="right" location="-1" />
-    <xacro:include filename="$(find heron_vortex_description)/urdf/accessories.urdf.xacro" />
+    <xacro:include filename="$(find asv_description)/urdf/accessories.urdf.xacro" />
     <!-- Optional custom includes. -->
     <xacro:include filename="$(optenv HERON_URDF_EXTRAS empty.urdf)" />

File: asv_description/urdf/heron.urdf.xacro (robot description, xacro)
@@ -30,6 +30,6 @@
   <xacro:arg name="suffix_ns" default="$(arg namespace)"/>
   <!-- Include the ROV macro file -->
-  <xacro:include filename="$(find heron_vortex_description)/urdf/base.xacro"/>
-  <xacro:include filename="$(find heron_vortex_description)/urdf/gazebo.xacro"/>
+  <xacro:include filename="$(find asv_description)/urdf/base.xacro"/>
+  <xacro:include filename="$(find asv_description)/urdf/gazebo.xacro"/>
   <!-- Create the heron -->
   <xacro:heron_base namespace="$(arg suffix_ns)">

File: asv_description/urdf/snippets.xacro (robot description, xacro)
@@ -15,5 +15,5 @@
       <visual>
         <geometry>
-          <mesh filename="package://heron_vortex_description/meshes/prop.dae" scale="1 1 1" />
+          <mesh filename="package://asv_description/meshes/prop.dae" scale="1 1 1" />
         </geometry>
       </visual>
